File: Modules/Common Template/Current_Version/Kicad/template_core_easyphi.sch (KiCad schematic (older format))
At the start: 128 parts, among them J1 JTAG_CONNEC, J2 DM3D-SF(AS), P1 CONN_8, Q1 MOS_P, Q2 FDD8780, Q3 FDD8780, U1 MAX5924D, U10 2-1825027-0, U12 TE-5650478-5, U15 TROU_FIX, U16 TROU_FIX, U2 MAX5925D, U23 RLP1-600-800, U3 24LC64, U4 USBLC6-2, U5 TPS7A4901, U51 CARD_BORDER, U52 CARD_BORDER, U53 CARD_BORDER, U54 CARD_BORDER, U6 AOZ1280, U7 SAM3X8E, U8 SN74LVC2G240DCTR, U9 SN65LVDM176DGK, X1 12MHz, X2 32.768KHz

Commit message: update on template
Changed lines of the file:
@@
 Sheet 2 2
 Title ""
-Date "8 oct 2013"
+Date "18 oct 2013"
 Rev ""
 Comp ""
@@
 Text Notes 12200 10950 0    59   ~ 0
 Easy-phi module template - CERN OHL
+$Comp
+L LOGO #G?
+U 1 1 526179E3
+P 15200 10150
+F 0 "#G?" H 15200 9650 60  0001 C CNN
+F 1 "LOGO" H 15200 10650 60  0001 C CNN
+F 2 "" H 15200 10150 60  0000 C CNN
+F 3 "" H 15200 10150 60  0000 C CNN
+	1    15200 10150
+	1    0    0    -1
+$EndComp
 $EndSCHEMATC
