File: Modules/Common Template/Current_Version/Kicad/top_level_easyphi.kicad_pcb (KiCad board)
At the start: 4 copper layers, 165 parts, among them J1 JTAG_CONNEC, J2 DM3D-SF(AS), P1 CONN_8, Q1 MOS_P, Q2 FDD8780, Q3 FDD8780, U1 MAX5924D, U10 2-1825027-0, U11 RLP1-600-800, U12 TE-5650478-5, U15 TROU_FIX, U16 TROU_FIX, U17 RLP1-600-800, U18 RLP1-600-800, U19 RLP1-600-800, U2 MAX5925D, U20 RLP1-600-800, U21 RLP1-600-800, U22 CONNEC_QMA_ANO_2622-4035, U23 RLP1-600-800, U24 CONNEC_QMA_ANO_2622-4035, U25 CONNEC_QMA_ANO_2622-4035, U26 CONNEC_QMA_ANO_2622-4035, U27 CONNEC_QMA_ANO_2622-4035, U28 CONNEC_QMA_ANO_2622-4035, U3 24LC64, U4 USBLC6-2, U5 TPS7A4901, U51 CARD_BORDER, U52 CARD_BORDER, U53 CARD_BORDER, U54 CARD_BORDER, U6 AOZ1280, U7 SAM3X8E, U8 SN74LVC2G240DCTR, U9 SN65LVDM176DGK, X1 12MHz, X2 32.768KHz

Commit message: update on template
Parts:
- added VAL: Logo, Logo, F.Cu at (161.5, 68.2)
Routing:
- net (no net): track 0.00 -> 77.5 mm
- net GND: track 484.3 -> 477.9 mm, vias 71 -> 133
- net /template core easyphi/USR_BUTTN: track 200.2 -> 199.2 mm
Other:
- board text added: "Arduino Programming Header"
- board text added: "JTAG"
- board text added: "Licensed under CERN OHL V1.2"
- board text added: "University of Geneva GAP-Optique Switzerland"
- board text added: "[TODO Module Name V1.0]"
- board text added: "www.easy-phi.ch"
- board text removed: "CERN OHL"
- board text removed: "DNP"
- board text removed: "University of Geneva GAP-Optique Proto Board Easy-Phi Version 2.0 [c] 2013 UniGe"
