File: Rack/Kicad/small_rack.sch (KiCad schematic (older format))
At the start: 63 parts, among them J1 MOLEX_0015244745, J1001 HOLE_BP, J1002 HOLE_BP, J1003 HOLE_BP, J1004 HOLE_BP, J1005 HOLE_BP, J1006 HOLE_BP, J1007 HOLE_BP, J1008 HOLE_BP, J1009 HOLE_BP, J1010 HOLE_BP, J1011 HOLE_BP, J1012 HOLE_BP, J1013 HOLE_BP, J1014 HOLE_BP, J1015 HOLE_BP, J1016 HOLE_BP, J1017 HOLE_BP, J1018 HOLE_BP, J1019 HOLE_BP, J1020 HOLE_BP, J1021 SLIDER, J1022 SLIDER, J2 USB_CONNEC, U1 USB_CONNEC, U10 SN65LVDM176DGK, U2 TE-8-1393640-3, U25 CUBIEBOARD, U3 TE-8-1393640-3, U4 R-535.0PA, U5 MAX1685, U6 TE-8-1393640-3, U7 TE-8-1393640-3, U8 TE-8-1393640-3, U9 FOX924B

Commit message: Logo on rack
Parts:
- added B1: LICENCE_CERN, ~, symbol LICENCE_CERN
- added B2: LOGO, ~, symbol LOGO
Other:
- note added: "SLOT 1"
- note added: "SLOT 2"
- note added: "SLOT 3"
- note added: "SLOT 4"
- note added: "SLOT 5"
- note removed: "Rack schematics - CERN OHL LICENSE"
- moved on the sheet: C1, C10, C11, C12, C13, C2, C3, C4, C5, C53, C6, C7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
