File: Modules/Common Template/Current_Version/github/Kicad/template_core_easyphi.sch (KiCad schematic (older format))
At the start: 128 parts, among them J1 JTAG_CONNEC, J2 DM3D-SF(AS), P1 CONN_8, Q1 MOS_P, Q2 FDD8780, Q3 FDD8780, U1 MAX5924D, U10 2-1825027-0, U12 TE-5650478-5, U15 TROU_FIX, U16 TROU_FIX, U2 MAX5925D, U23 RLP1-600-800, U3 24LC64, U4 USBLC6-2, U5 TPS7A4901, U51 CARD_BORDER, U52 CARD_BORDER, U53 CARD_BORDER, U54 CARD_BORDER, U6 AOZ1280, U7 SAM3X8E, U8 SN74LVC2G240DCTR, U9 SN65LVDM176DGK, X1 12MHz, X2 32.768KHz

Commit message: final update common template
Parts:
- added B3: LICENCE_CERN, ~, symbol LICENCE_CERN
- added B4: LOGO, ~, symbol LOGO
Other:
- note removed: "Easy-phi module template - CERN OHL"
- moved on the sheet: C17, C18, C19, C21, C22, C23, C24, C27, C28, C29, C30, C31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
