File: Modules/Common Template/Current_Version/github/Kicad/top_level_easyphi.sch (KiCad schematic (older format))
At the start: 37 parts, among them U11 RLP1-600-800, U17 RLP1-600-800, U18 RLP1-600-800, U19 RLP1-600-800, U20 RLP1-600-800, U21 RLP1-600-800, U22 CONNEC_QMA_ANO_2622-4035, U24 CONNEC_QMA_ANO_2622-4035, U25 CONNEC_QMA_ANO_2622-4035, U26 CONNEC_QMA_ANO_2622-4035, U27 CONNEC_QMA_ANO_2622-4035, U28 CONNEC_QMA_ANO_2622-4035

Commit message: final update common template
Parts:
- added B1: LICENCE_CERN, ~, symbol LICENCE_CERN
- added B2: LOGO, ~, symbol LOGO
Other:
- note removed: "Easy-phi module template - CERN OHL"
Changed lines of the file:
@@
 encoding utf-8
 Sheet 1 2
-Title ""
-Date "18 oct 2013"
-Rev ""
-Comp ""
+Title "Easy-phi Module Template"
+Date "23 oct 2013"
+Rev "1.0"
+Comp "University of Geneva                       www.easy-phi.ch"
 Comment1 ""
 Comment2 ""
@@
 $EndDescr
 $Comp
-L GND #PWR01
+L GND #PWR17
 U 1 1 501BE141
 P 13000 1950
-F 0 "#PWR01" H 13000 1950 30  0001 C CNN
+F 0 "#PWR17" H 13000 1950 30  0001 C CNN
 F 1 "GND" H 13000 1880 30  0001 C CNN
 F 2 "" H 13000 1950 60  0001 C CNN
@@
 $EndComp
 $Comp
-L +3.3V #PWR02
+L +3.3V #PWR5
 U 1 1 501FC859
 P 8150 1550
-F 0 "#PWR02" H 8150 1510 30  0001 C CNN
+F 0 "#PWR5" H 8150 1510 30  0001 C CNN
 F 1 "+3.3V" H 8150 1660 30  0000 C CNN
 F 2 "" H 8150 1550 60  0001 C CNN
@@
 $EndComp
 $Comp
-L +3.3V #PWR03
+L +3.3V #PWR6
 U 1 1 501FC94B
 P 8150 2350
-F 0 "#PWR03" H 8150 2310 30  0001 C CNN
+F 0 "#PWR6" H 8150 2310 30  0001 C CNN
 F 1 "+3.3V" H 8150 2460 30  0000 C CNN
 F 2 "" H 8150 2350 60  0001 C CNN
@@
 $EndComp
 $Comp
-L +3.3V #PWR04
+L +3.3V #PWR7
 U 1 1 501FC963
 P 8150 3150
-F 0 "#PWR04" H 8150 3110 30  0001 C CNN
+F 0 "#PWR7" H 8150 3110 30  0001 C CNN
 F 1 "+3.3V" H 8150 3260 30  0000 C CNN
 F 2 "" H 8150 3150 60  0001 C CNN
@@
 $EndComp
 $Comp
-L +3.3V #PWR05
+L +3.3V #PWR8
 U 1 1 501FC975
 P 8150 3950
-F 0 "#PWR05" H 8150 3910 30  0001 C CNN
+F 0 "#PWR8" H 8150 3910 30  0001 C CNN
 F 1 "+3.3V" H 8150 4060 30  0000 C CNN
 F 2 "" H 8150 3950 60  0001 C CNN
@@
 $EndComp
 $Comp
-L GND #PWR06
+L GND #PWR11
 U 1 1 501FCC85
 P 10600 1650
-F 0 "#PWR06" H 10600 1650 30  0001 C CNN
+F 0 "#PWR11" H 10600 1650 30  0001 C CNN
 F 1 "GND" H 10600 1580 30  0001 C CNN
 F 2 "" H 10600 1650 60  0001 C CNN
@@
 R5 = ((Itriplow * 0.03) + 4.7mV) / 37uA\nSlew rate set to max 3.3V/ms
 Wire Notes Line
-	11850 8500 14200 8500
+	7600 8700 9950 8700
 Wire Notes Line
-	14200 8500 14200 9800
+	9950 8700 9950 10000
 Wire Notes Line
-	14200 8800 11850 8800
+	9950 9000 7600 9000
 Wire Notes Line
-	11850 8500 11850 9800
-Text Notes 12150 8700 0    60   ~ 0
+	7600 8700 7600 10000
+Text Notes 7900 8900 0    60   ~ 0
 ABOUT THE POWER SUPPLY SYMBOLS
 $Comp
-L +12V #PWR07
+L +12V #PWR1
 U 1 1 51B87547
-P 12050 9000
-F 0 "#PWR07" H 12050 8950 20  0001 C CNN
-F 1 "+12V" H 12050 9100 30  0000 C CNN
-F 2 "" H 12050 9000 60  0000 C CNN
-F 3 "" H 12050 9000 60  0000 C CNN
-	1    12050 9000
-	1    0    0    -1
-$EndComp
-$Comp
-L +5V #PWR08
+P 7800 9200
+F 0 "#PWR1" H 7800 9150 20  0001 C CNN
+F 1 "+12V" H 7800 9300 30  0000 C CNN
+F 2 "" H 7800 9200 60  0000 C CNN
+F 3 "" H 7800 9200 60  0000 C CNN
+	1    7800 9200
+	1    0    0    -1
+$EndComp
+$Comp
+L +5V #PWR2
 U 1 1 51B87556
-P 12050 9250
-F 0 "#PWR08" H 12050 9340 20  0001 C CNN
-F 1 "+5V" H 12050 9340 30  0000 C CNN
-F 2 "" H 12050 9250 60  0000 C CNN
-F 3 "" H 12050 9250 60  0000 C CNN
-	1    12050 9250
-	1    0    0    -1
-$EndComp
-$Comp
-L +3.3V #PWR09
+P 7800 9450
+F 0 "#PWR2" H 7800 9540 20  0001 C CNN
+F 1 "+5V" H 7800 9540 30  0000 C CNN
+F 2 "" H 7800 9450 60  0000 C CNN
+F 3 "" H 7800 9450 60  0000 C CNN
+	1    7800 9450
+	1    0    0    -1
+$EndComp
+$Comp
+L +3.3V #PWR3
 U 1 1 51B87565
-P 12050 9500
-F 0 "#PWR09" H 12050 9460 30  0001 C CNN
-F 1 "+3.3V" H 12050 9610 30  0000 C CNN
-F 2 "" H 12050 9500 60  0000 C CNN
-F 3 "" H 12050 9500 60  0000 C CNN
-	1    12050 9500
-	1    0    0    -1
-$EndComp
-$Comp
-L +3.3VADC #PWR010
+P 7800 9700
+F 0 "#PWR3" H 7800 9660 30  0001 C CNN
+F 1 "+3.3V" H 7800 9810 30  0000 C CNN
+F 2 "" H 7800 9700 60  0000 C CNN
+F 3 "" H 7800 9700 60  0000 C CNN
+	1    7800 9700
+	1    0    0    -1
+$EndComp
+$Comp
+L +3.3VADC #PWR4
 U 1 1 51B8772D
-P 12050 9750
-F 0 "#PWR010" H 12050 9870 20  0001 C CNN
-F 1 "+3.3VADC" H 12050 9840 30  0000 C CNN
-F 2 "" H 12050 9750 60  0000 C CNN
-F 3 "" H 12050 9750 60  0000 C CNN
-	1    12050 9750
-	1    0    0    -1
-$EndComp
-Text Notes 12300 8950 0    40   ~ 0
+P 7800 9950
+F 0 "#PWR4" H 7800 10070 20  0001 C CNN
+F 1 "+3.3VADC" H 7800 10040 30  0000 C CNN
+F 2 "" H 7800 9950 60  0000 C CNN
+F 3 "" H 7800 9950 60  0000 C CNN
+	1    7800 9950
+	1    0    0    -1
+$EndComp
+Text Notes 8050 9150 0    40   ~ 0
 is the 12V filtered coming from the backplane (MAX 4A)\nset R5 according to the max current you'll have
-Text Notes 12300 9200 0    40   ~ 0
+Text Notes 8050 9400 0    40   ~ 0
 is the 5V filtered coming from the backplane (MAX 0.5A)
-Text Notes 12300 9450 0    40   ~ 0
+Text Notes 8050 9650 0    40   ~ 0
 is a 3.3V generated from this 5V by a stepdown\nused by template_core chips
-Text Notes 12300 9700 0    40   ~ 0
+Text Notes 8050 9900 0    40   ~ 0
 is a 3.3V generated from the 5V by a LDO\nused by the uC ADC
 Wire Notes Line
-	11850 9050 14200 9050
+	7600 9250 9950 9250
 Wire Notes Line
-	11850 9300 14200 9300
+	7600 9500 9950 9500
 Wire Notes Line
-	11850 9550 14200 9550
+	7600 9750 9950 9750
 Wire Notes Line
-	11850 9800 14200 9800
+	7600 10000 9950 10000
 Wire Wire Line
 	2950 9400 3100 9400
@@
 $EndComp
 $Comp
-L +3.3V #PWR011
+L +3.3V #PWR9
 U 1 1 5232ED9B
 P 8150 4750
-F 0 "#PWR011" H 8150 4710 30  0001 C CNN
+F 0 "#PWR9" H 8150 4710 30  0001 C CNN
 F 1 "+3.3V" H 8150 4860 30  0000 C CNN
 F 2 "" H 8150 4750 60  0001 C CNN
@@
 $EndComp
 $Comp
-L +3.3V #PWR012
+L +3.3V #PWR10
 U 1 1 5232F96D
 P 8150 5550
-F 0 "#PWR012" H 8150 5510 30  0001 C CNN
+F 0 "#PWR10" H 8150 5510 30  0001 C CNN
 F 1 "+3.3V" H 8150 5660 30  0000 C CNN
 F 2 "" H 8150 5550 60  0001 C CNN
@@
 	9750 5600 10000 5600
 $Comp
-L GND #PWR013
+L GND #PWR12
 U 1 1 52331404
 P 10600 2450
-F 0 "#PWR013" H 10600 2450 30  0001 C CNN
+F 0 "#PWR12" H 10600 2450 30  0001 C CNN
 F 1 "GND" H 10600 2380 30  0001 C CNN
 F 2 "" H 10600 2450 60  0001 C CNN
@@
 	10650 2500 10700 2500
 $Comp
-L GND #PWR014
+L GND #PWR13
 U 1 1 5233150E
 P 10600 3250
-F 0 "#PWR014" H 10600 3250 30  0001 C CNN
+F 0 "#PWR13" H 10600 3250 30  0001 C CNN
 F 1 "GND" H 10600 3180 30  0001 C CNN
 F 2 "" H 10600 3250 60  0001 C CNN
@@
 	10650 3300 10700 3300
 $Comp
-L GND #PWR015
+L GND #PWR14
 U 1 1 52331618
 P 10600 4050
-F 0 "#PWR015" H 10600 4050 30  0001 C CNN
+F 0 "#PWR14" H 10600 4050 30  0001 C CNN
 F 1 "GND" H 10600 3980 30  0001 C CNN
 F 2 "" H 10600 4050 60  0001 C CNN
@@
 	10650 4100 10700 4100
 $Comp
-L GND #PWR016
+L GND #PWR15
 U 1 1 52331722
 P 10600 4850
-F 0 "#PWR016" H 10600 4850 30  0001 C CNN
+F 0 "#PWR15" H 10600 4850 30  0001 C CNN
 F 1 "GND" H 10600 4780 30  0001 C CNN
 F 2 "" H 10600 4850 60  0001 C CNN
@@
 	10650 4900 10700 4900
 $Comp
-L GND #PWR017
+L GND #PWR16
 U 1 1 5233182C
 P 10600 5650
-F 0 "#PWR017" H 10600 5650 30  0001 C CNN
+F 0 "#PWR16" H 10600 5650 30  0001 C CNN
 F 1 "GND" H 10600 5580 30  0001 C CNN
 F 2 "" H 10600 5650 60  0001 C CNN
@@
 	10650 5700 10700 5700
 $Comp
-L GND #PWR018
+L GND #PWR18
 U 1 1 523331B2
 P 13000 2750
-F 0 "#PWR018" H 13000 2750 30  0001 C CNN
+F 0 "#PWR18" H 13000 2750 30  0001 C CNN
 F 1 "GND" H 13000 2680 30  0001 C CNN
 F 2 "" H 13000 2750 60  0001 C CNN
@@
 Connection ~ 13000 2550
 $Comp
-L GND #PWR019
+L GND #PWR19
 U 1 1 523332C0
 P 13000 3550
-F 0 "#PWR019" H 13000 3550 30  0001 C CNN
+F 0 "#PWR19" H 13000 3550 30  0001 C CNN
 F 1 "GND" H 13000 3480 30  0001 C CNN
 F 2 "" H 13000 3550 60  0001 C CNN
@@
 Connection ~ 13000 3350
 $Comp
-L GND #PWR020
+L GND #PWR20
 U 1 1 5233500D
 P 13000 4350
-F 0 "#PWR020" H 13000 4350 30  0001 C CNN
+F 0 "#PWR20" H 13000 4350 30  0001 C CNN
 F 1 "GND" H 13000 4280 30  0001 C CNN
 F 2 "" H 13000 4350 60  0001 C CNN
@@
 Connection ~ 13000 4150
 $Comp
-L GND #PWR021
+L GND #PWR21
 U 1 1 52335406
 P 13000 5150
-F 0 "#PWR021" H 13000 5150 30  0001 C CNN
+F 0 "#PWR21" H 13000 5150 30  0001 C CNN
 F 1 "GND" H 13000 5080 30  0001 C CNN
 F 2 "" H 13000 5150 60  0001 C CNN
@@
 Connection ~ 13000 4950
 $Comp
-L GND #PWR022
+L GND #PWR22
 U 1 1 52335514
 P 13000 5950
-F 0 "#PWR022" H 13000 5950 30  0001 C CNN
+F 0 "#PWR22" H 13000 5950 30  0001 C CNN
 F 1 "GND" H 13000 5880 30  0001 C CNN
 F 2 "" H 13000 5950 60  0001 C CNN
@@
 	13300 5650 13000 5650
 Connection ~ 13000 5750
-Text Notes 12200 10950 0    59   ~ 0
-Easy-phi module template - CERN OHL
-$Comp
-L LOGO #G?
-U 1 1 5261604F
-P 15200 10150
-F 0 "#G?" H 15200 9650 60  0001 C CNN
-F 1 "LOGO" H 15200 10650 60  0001 C CNN
-F 2 "" H 15200 10150 60  0000 C CNN
-F 3 "" H 15200 10150 60  0000 C CNN
-	1    15200 10150
-	1    0    0    -1
-$EndComp
+$Comp
+L LICENCE_CERN B1
+U 1 1 5267FE20
+P 11850 10500
+F 0 "B1" H 11916 11547 60  0001 C CNN
+F 1 "LICENCE_CERN" H 13566 11547 60  0001 C CNN
+F 2 "~" H 12316 10647 60  0000 C CNN
+F 3 "~" H 12316 10647 60  0000 C CNN
+	1    11850 10500
+	1    0    0    -1
+$EndComp
+$Comp
+L LOGO B2
+U 1 1 52680405
+P 15050 10000
+F 0 "B2" H 15050 9500 60  0001 C CNN
+F 1 "LOGO" H 15050 10500 60  0001 C CNN
+F 2 "~" H 15050 10000 60  0000 C CNN
+F 3 "~" H 15050 10000 60  0000 C CNN
+	1    15050 10000
+	1    0    0    -1
+$EndComp
