File: Modules/High-speed Logic gate/Current Version/github/Kicad/LogicGate.sch (KiCad schematic (older format))
At the start: 88 parts, among them U13 LM7321MF, U14 LM7321MF, U29 SY89854U, U30 SY89854U, U31 MC100LVEP05DTG, U32 MC100LVEP05DTG, U33 AOZ1280, U34 SY89540U, U35 SY89850U, U36 SY89850U, U37 SY89850U, U38 SY89850U

Commit message: update firmwares
Parts:
- C16, C20: value 1nF -> 100nF
Changed lines of the file:
@@
 Sheet 3 9
 Title "High-speed Logic Gate"
-Date "6 dec 2013"
+Date "15 apr 2014"
 Rev "1.0"
 Comp "University of Geneva             www.easy-phi.ch"
@@
 P 2500 3150
 F 0 "C16" H 2500 3250 40  0000 L CNN
-F 1 "1nF" H 2506 3065 40  0000 L CNN
+F 1 "100nF" H 2506 3065 40  0000 L CNN
 F 2 "~" H 2538 3000 30  0000 C CNN
 F 3 "~" H 2500 3150 60  0000 C CNN
@@
 P 2500 9400
 F 0 "C20" H 2500 9500 40  0000 L CNN
-F 1 "1nF" H 2506 9315 40  0000 L CNN
+F 1 "100nF" H 2506 9315 40  0000 L CNN
 F 2 "~" H 2538 9250 30  0000 C CNN
 F 3 "~" H 2500 9400 60  0000 C CNN
